File: KiCAD/handheldAerosolSensor/handheldAerosolSensor.kicad_sch (KiCad schematic)
At the start: 15 parts, among them J1 BAT IN (3.7v), J2 PUSH BUTTON, J3 MCU, J4 MCU, J5 DC/DC Bootser, J6 PWR OUT 5volt, Q1 IRF4905, Q2 2N7000

Commit message: Many inprovements
Parts:
- removed A1: Arduino_Nano_v3.x, Module:Arduino_Nano, symbol MCU_Module:Arduino_Nano_v3.x
- removed J1: BAT IN (3.7v), symbol Connector:Conn_01x02_Socket
- removed J2: PUSH BUTTON, symbol Connector:Conn_01x02_Socket
- removed J3: MCU, symbol Connector:Conn_01x04_Socket
- removed J4: MCU, symbol Connector:Conn_01x04_Pin
- removed J6: PWR OUT 5volt, symbol Connector:Conn_01x02_Socket
- added BT1: BH-18650-PC, BH-18650-PC:BAT_BH-18650-PC, symbol MyNewLibrary:BH-18650-PC
- added C2: 0.1uF, Capacitor_SMD:C_1206_3216Metric_Pad1.33x1.80mm_HandSolder, symbol Device:C_Small
- added J1: I2C 3v3, Connector_JST:JST_XH_B4B-XH-A_1x04_P2.50mm_Vertical, symbol Connector:Conn_01x04_Pin
- added J2: ePaper, Connector_JST:JST_XH_B8B-XH-A_1x08_P2.50mm_Vertical, symbol Connector:Conn_01x08_Pin
- added J3: SPS30, Connector_JST:JST_XH_B5B-XH-A_1x05_P2.50mm_Vertical, symbol Connector:Conn_01x05_Pin
- added J4: BME/P280, Connector_PinSocket_2.54mm:PinSocket_1x06_P2.54mm_Vertical, symbol Connector:Conn_01x06_Pin
- added LS1: PIEZO, MyNewLibrary:XDCR_CPI-148-24-90T-67, symbol MyNewLibrary:CPI-148-24-90T-67
- added Q3: BSS138, Package_TO_SOT_SMD:SOT-23, symbol Transistor_FET:2N7000
- added R4, R5, R9: 100k, Resistor_SMD:R_1206_3216Metric_Pad1.30x1.75mm_HandSolder, symbol Device:R
- added R6: 10R-220R, Resistor_SMD:R_1206_3216Metric_Pad1.30x1.75mm_HandSolder, symbol Device:R
- added R7: 1k, Resistor_SMD:R_1206_3216Metric_Pad1.30x1.75mm_HandSolder, symbol Device:R
- added R8: 2k2, Resistor_SMD:R_1206_3216Metric_Pad1.30x1.75mm_HandSolder, symbol Device:R
- added SW1: PWR, Button_Switch_THT:SW_PUSH_6mm_H4.3mm, symbol Switch:SW_Push
- added U1: ~, MyNewLibrary:TP4056_USB-Charger_Board, symbol MyNewLibrary:TP4056Module
- added U2: Mini DC-DC Convertor, MyNewLibrary:Mini DC-DC Boost Convertor, symbol MyNewLibrary:Mini_DC-DC_Boost_Convertor
- added U3: ESP32-DEVKIT-V1 30pin, MyNewLibrary:MODULE_ESP32_DEVKIT_V1_30pin, symbol MyNewLibrary:ESP32-DEVKIT-V1-30pin
- C1: footprint (none) -> Capacitor_SMD:C_1206_3216Metric_Pad1.33x1.80mm_HandSolder
- D1: renamed from D2; footprint (none) -> Diode_SMD:D_1206_3216Metric_Pad1.42x1.75mm_HandSolder
- D2: renamed from D1; footprint (none) -> Diode_SMD:D_1206_3216Metric_Pad1.42x1.75mm_HandSolder
- J5: value DC/DC Bootser -> Ext.Sw; footprint (none) -> Connector_JST:JST_XH_B2B-XH-A_1x02_P2.50mm_Vertical
- Q1: value IRF4905 -> AO3401; footprint Package_TO_SOT_THT:TO-220-3_Vertical -> Package_TO_SOT_SMD:SOT-23
- Q2: value 2N7000 -> BSS138; footprint Package_TO_SOT_THT:TO-92_Inline -> Package_TO_SOT_SMD:SOT-23
- R1: footprint (none) -> Resistor_SMD:R_1206_3216Metric_Pad1.30x1.75mm_HandSolder
- R2: renamed from R3; value 220 -> 10R-220R; footprint (none) -> Resistor_SMD:R_1206_3216Metric_Pad1.30x1.75mm_HandSolder
- R3: renamed from R2; footprint (none) -> Resistor_SMD:R_1206_3216Metric_Pad1.30x1.75mm_HandSolder
Connections:
- net GND: now also BT1.N, C2.2, J1.1 (Pin_1), J2.7 (Pin_7), J3.1 (Pin_1), J3.2 (Pin_2), J4.2 (Pin_2), Q3.1 (S), R5.2, R9.2, SW1.1, U1.3 (Out-), U2.1 (In-), U2.3 (Out-), U3.2 (GND), U3.29 (GND)
- net at J5.1 (Pin_1): now also D1.1 (K), D2.1 (K), SW1.2; no longer Q1.2 (D)
- net BATT: now reaches Q1.3 (S), R1.1
- net BATT: now also BT1.P, U1.4 (Out+)
- net LATCH: now reaches R2.2
- net LATCH: now also U3.23 (D25)
- net SWITCH: now reaches D2.2 (A)
- net SWITCH: now also U3.22 (D33)
- new net: LS1.N, R6.1, R8.2
- new net: Q3.3 (D), R6.2
- new net: Q3.2 (G), R7.1, R9.1
- new net: C2.1, R4.2, R5.1, U3.19 (D34)
- new net +5v: J3.5 (Pin_5), LS1.P, R8.1, U2.4 (Out+), U3.30 (VIN)
- new net 3v3: J1.2 (Pin_2), J2.8 (Pin_8), J4.1 (Pin_1), U3.1 (3V3)
- new net BATT-SW: Q1.2 (D), R4.1, U2.2 (In+)
- new net BUZZER: R7.2, U3.26 (D14)
- new net EPD_BUSY: J2.1 (Pin_1), U3.21 (D32)
- new net EPD_CS: J2.4 (Pin_4), U3.25 (D27)
- new net EPD_DC: J2.3 (Pin_3), U3.10 (D19)
- new net EPD_MOSI(DIN): J2.6 (Pin_6), U3.15 (D23)
- new net EPD_RST: J2.2 (Pin_2), U3.28 (D13)
- new net EPS_SCK: J2.5 (Pin_5), U3.9 (D18)
- new net RX2: U3.6 (RX2)
- new net SCL: J1.4 (Pin_4), J3.3 (Pin_3), J4.3 (Pin_3), J4.4 (Pin_4), U3.14 (D22)
- new net SDA: J1.3 (Pin_3), J3.4 (Pin_4), U3.11 (D21)
- new net TX2: U3.7 (TX2)
- no-connect marks 0 -> 16
Other:
- note added: "1=Vcc=Black"
- note added: "5=GND=Orange"
- note added: "BSS138"
- note added: "Rood"
- note added: "White"
- note added: "Yellow"
- note removed: "DC/DC Booster"
- company: (none) -> By Willem Aandewiel
- title: (none) -> handheldAerosolSensor
- moved on the sheet: D2, R2
